File: TRIATLON/HARDWARE/KICAD_MAIN/PLACA_DE_SENSORES/SENSORES (1).kicad_pcb (KiCad board)
At the start: 2 copper layers, 108 parts, among them J1 Cable_PAD, J2 Conn_01x10_Socket, J3 Cable_PAD, U1 TCRT5000, U10 TCRT5000, U3 TCRT5000, U4 TCRT5000, U5 TCRT5000, U6 TCRT5000, U8 TCRT5000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

Commit message: actualizado
Parts:
- J1, J3: footprint EESTN5 huellas:Tornillo_M3_8mm -> EESTN5:Tornillo_M3_8mm
