File: TRIATLON/HARDWARE/KICAD_MAIN/PLACA_DE_SENSORES/SENSORES (1).kicad_sch (KiCad schematic)
At the start: 27 parts, among them J1 Cable_PAD, J2 Conn_01x10_Socket, J3 Cable_PAD, U1 TCRT5000, U10 TCRT5000, U3 TCRT5000, U4 TCRT5000, U5 TCRT5000, U6 TCRT5000, U8 TCRT5000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

Commit message: actualizado
Parts:
- J1, J3: footprint EESTN5 huellas:Tornillo_M3_8mm -> EESTN5:Tornillo_M3_8mm
Changed lines of the file:
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@@
 			)
 		)
-		(property "Footprint" "EESTN5 huellas:Tornillo_M3_8mm"
+		(property "Footprint" "EESTN5:Tornillo_M3_8mm"
 			(at 163.83 110.49 0)
 			(effects
@@
 			)
 		)
-		(property "Footprint" "EESTN5 huellas:Tornillo_M3_8mm"
+		(property "Footprint" "EESTN5:Tornillo_M3_8mm"
 			(at 163.83 105.41 0)
 			(effects
