File: TRIATLON/HARDWARE/KICAD_MAIN/PLACA_PRINCIPAL/Triatron (1).kicad_pcb (KiCad board)
At the start: 2 copper layers, 26 parts, among them J1 Screw_Terminal_01x02, J10 HC-04, J11 HC-04, J12 HC-04, J13 Conn_01x06_Pin, J2 Conn_01x10_Pin, J3 Conn_01x04_Pin, J4 Conn_01x06_Pin, J5 infrarrojo, J6 Conn_01x04_Pin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

Commit message: actualizado
Parts:
- removed J6: Conn_01x04_Pin, Connector_PinHeader_2.54mm:PinHeader_1x04_P2.54mm_Vertical
- added J14: Screw_Terminal_01x02, TerminalBlock_MetzConnect:TerminalBlock_MetzConnect_Type055_RT01502HDWU_1x02_P5.00mm_Horizontal, F.Cu at (146.5, 102.6)
- added J15: Screw_Terminal_01x02, TerminalBlock_MetzConnect:TerminalBlock_MetzConnect_Type055_RT01502HDWU_1x02_P5.00mm_Horizontal, F.Cu at (163.1, 102.6)
- J3: footprint Connector_PinSocket_2.54mm:PinSocket_1x04_P2.54mm_Vertical -> Connector_PinHeader_2.54mm:PinHeader_1x04_P2.54mm_Vertical
- R10: value R -> 220
- R3: value R -> 1k
- R4: value R -> 2k
- moved R9 113.2 mm to (93.6, 107.5), turned to 90 degrees
- moved R8 110.3 mm to (97.1, 107.5), turned to 90 degrees
- moved R7 103.8 mm to (104.5, 107.5), turned to 90 degrees
- moved R6 101.2 mm to (108.0, 107.5), turned to 90 degrees
- moved R5 95.5 mm to (115.0, 107.3), turned to 90 degrees
- moved R2 93.7 mm to (118.0, 107.3), turned to 90 degrees
- moved R3 85.0 mm to (129.0, 107.5), turned to 90 degrees
- moved J12 70.4 mm to (100.6, 112.5), turned to 180 degrees
- moved R4 67.9 mm to (125.5, 99.8), turned to -90 degrees
- moved J11 55.3 mm to (111.5, 112.5), turned to 180 degrees
- moved J10 41.3 mm to (121.5, 112.5), turned to 180 degrees
- moved R10 36.2 mm to (140.0, 94.4), turned to -90 degrees
- moved J1 32.0 mm to (162.0, 84.5), turned to 90 degrees
- moved J3 31.6 mm to (153.0, 94.5), turned to 90 degrees
- moved D1 28.0 mm to (140.0, 87.5), turned to -90 degrees
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Connections:
- J1 pad 1: OUT+ -> VCC
- J1 pad 2: IN- -> GND
- J10 pad 1: IN+ -> OUT+
- J10 pad 4: GND -> OUT-
- J11 pad 1: IN+ -> OUT+
- J11 pad 4: GND -> OUT-
- J12 pad 1: IN+ -> OUT+
- J12 pad 4: GND -> OUT-
- J13 pad 3: EN-L 2 -> EN
- J13 pad 4: EN-R 2 -> EN
- J13 pad 5: GND -> OUT-
- J13 pad 6: IN+ -> OUT+
- J2 pad 10: GND -> OUT-
- J2 pad 9: IN+ -> OUT+
- J3 pad 2: IN- -> OUT-
- J3 pad 4: IN+ -> VCC
- J4 pad 3: EN-L -> EN
- J4 pad 4: EN-R -> EN
- J4 pad 5: GND -> OUT-
- J4 pad 6: IN+ -> OUT+
- J5 pad 1: IN+ -> OUT+
- J5 pad 2: GND -> OUT-
- J7 pad 1: IN+ -> OUT+
- J7 pad 2: GND -> OUT-
- J8 pad 1: IN+ -> OUT+
- J8 pad 2: GND -> OUT-
- J9 pad 1: IN+ -> OUT+
- J9 pad 4: GND -> OUT-
- R10 pad 2: GND -> OUT-
- R4 pad 2: GND -> OUT-
- R5 pad 1: GND -> OUT-
- R7 pad 1: GND -> OUT-
- R9 pad 1: GND -> OUT-
- SW1 pad 1: GND -> OUT-
- SW1 pad 2: GND -> OUT-
- SW1 pad 3: SW2 -> SW1
- SW1 pad 4: SW1 -> SW2
- U2 pad 14: GND -> OUT-
- U2 pad 15: IN+ -> OUT+
- U2 pad 19: TRIG1 -> ECHO2
- U2 pad 20: ECHO1 -> ECHO3
- U2 pad 21: EN-R 2 -> unconnected-(U2-GPIO16-Pad21)
- U2 pad 22: EN-L 2 -> EN
- U2 pad 25: PWM-L -> ECHO4
- U2 pad 26: PWM-R -> PWM-L
- U2 pad 27: EN-L -> PWM-R
- U2 pad 28: EN-R -> unconnected-(U2-GPIO1-Pad28)
- U2 pad 29: ECHO2 -> unconnected-(U2-GPIO22-Pad29)
- U2 pad 4: ECHO4 -> ECHO1
- U2 pad 5: ECHO3 -> TRIG1
- U3 pad JP3-1: GND -> OUT-
- U3 pad JP3-2: IN+ -> OUT+
Routing:
- net OUT+: track 20.2 -> 243.6 mm
- net TRIG1: track 14.5 -> 73.6 mm
- net ECHO2: track 2.69 -> 55.6 mm
- net ECHO3: track 0.00 -> 47.3 mm
- net VCC: track 0.00 -> 42.2 mm
- net ECHO4: track 0.00 -> 39.9 mm
- net IN+: track 37.7 -> 0.00 mm
- net A2: track 31.8 -> 4.00 mm
- net EN: track 0.00 -> 27.7 mm
- net ECHO1: track 0.00 -> 27.0 mm
- net OUT-: track 0.00 -> 15.7 mm
- net D10: track 15.7 -> 24.9 mm
- net IN-: track 8.15 -> 0.00 mm
- net GND: track 38.4 -> 32.8 mm
- net EN-R: track 5.14 -> 0.00 mm
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- added copper zone on B.Cu, net OUT-
